File: hardware/1.3/watch.brd (EAGLE design)
At the start: 35.6 x 36.8 mm, 51 parts, among them J1 POGOPROG-WATCH, Q1 DMP2035U, Q2 NX3008PBK, Q3 NX7002AKA, Q4 NX3008NBK, U1 ATMEGA328P, U2 DS3231MZ+, U3 MCP73832T-2ACI/OT, U4 XC6206P252MR

Commit message: Schematic adjustments
D1 was ZLLS410, should be BAT60JFILM
Parts:
- D1: value ZLLS410 -> BAT60JFILM
Changed lines of the file:
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@@
 <attribute name="VALUE" x="59.40425" y="26.63825" size="0.4064" layer="27" ratio="10" rot="R180"/>
 </element>
-<element name="D1" library="zak" package="SOD-323" value="ZLLS410" x="56.8325" y="20.6375" smashed="yes" rot="MR90">
+<element name="D1" library="zak" package="SOD-323" value="BAT60JFILM" x="56.8325" y="20.6375" smashed="yes" rot="MR90">
 <attribute name="NAME" x="58.53125" y="22.3725" size="0.8128" layer="26" ratio="18" rot="MR270"/>
 <attribute name="VALUE" x="55.0405" y="19.5375" size="0.4064" layer="28" ratio="10" rot="MR90"/>
