File: hardware/1.3/watch.sch (EAGLE design)
At the start: 51 parts, among them J1 POGOPROG-WATCH, Q1 DMP2035U, Q2 NX3008PBK, Q3 NX7002AKA, Q4 NX3008NBK, U1 ATMEGA328P, U2 DS3231MZ+, U3 MCP73832T-2ACI/OT, U4 XC6206P252MR

Commit message: Schematic adjustments
D1 was ZLLS410, should be BAT60JFILM
Parts:
- D1: value ZLLS410 -> BAT60JFILM
Other:
- moved on the sheet: C7, D3, LED1, LED2, LS1, Q4, R4, RN2G$1
